File: sch/watch.kicad_pcb (KiCad board)
At the start: 4 copper layers, 19 parts, among them J1 eZ-FET, U1 MSP430FR2433IRGET, Y1 32.768kHz

Commit message: Updated the PCB
Parts:
- removed DIS1: HP-5082-7414, Package_DIP:DIP-12_W7.62mm_Socket_LongPads
- removed H1: SW1, MountingHole:MountingHole_3.2mm_M3_DIN965_Pad_TopBottom
- removed H2: SW2, MountingHole:MountingHole_3.2mm_M3_DIN965_Pad_TopBottom
- removed H3: SW3, MountingHole:MountingHole_3.2mm_M3_DIN965_Pad_TopBottom
- removed H4: SW4, MountingHole:MountingHole_3.2mm_M3_DIN965_Pad_TopBottom
- removed R4, R5, R6, R7: 1.5k, Resistor_SMD:R_0402_1005Metric_Pad0.72x0.64mm_HandSolder
- added C4: 12pF, Capacitor_SMD:C_0805_2012Metric_Pad1.18x1.45mm_HandSolder, F.Cu at (210.2, 97.6)
- added D1: 1N4148, Diode_SMD:D_SOD-323_HandSoldering, F.Cu at (207.4, 118.8)
- added DISP1: HP-5082-7414, Package_DIP:DIP-12_W8.89mm_SMDSocket_LongPads, F.Cu at (207.5, 109.5)
- added SW1: SW1, MountingHole:MountingHole_2.2mm_M2_DIN965_Pad_TopBottom, F.Cu at (193.5, 113.2)
- added SW2: SW2, MountingHole:MountingHole_2.2mm_M2_DIN965_Pad_TopBottom, F.Cu at (217.8, 99.2)
- added SW3: SW3, MountingHole:MountingHole_2.2mm_M2_DIN965_Pad_TopBottom, F.Cu at (217.8, 119.8)
- added SW4: SW4, MountingHole:MountingHole_2.2mm_M2_DIN965_Pad_TopBottom, F.Cu at (220.6, 115.6)
- added SW5: SW5, MountingHole:MountingHole_2.2mm_M2_DIN965_Pad_TopBottom, F.Cu at (220.6, 103.4)
- added U2: MSP430FR2433IRGET, Package_DFN_QFN:QFN-24-1EP_4x4mm_P0.5mm_EP2.7x2.7mm, F.Cu at (205.5, 100.0)
- BT1: footprint Battery:BatteryHolder_Keystone_3002_1x2032 -> Elektronika:BAT-HLD-001; moved to B.Cu
- C1: value 100nF low ESR -> 10uF*; footprint Capacitor_SMD:C_0603_1608Metric -> Capacitor_SMD:C_0805_2012Metric_Pad1.18x1.45mm_HandSolder
- C2: value 12pF -> 12pF*; footprint Capacitor_SMD:C_0402_1005Metric_Pad0.74x0.62mm_HandSolder -> Capacitor_SMD:C_0805_2012Metric_Pad1.18x1.45mm_HandSolder
- C3: footprint Capacitor_SMD:C_0402_1005Metric_Pad0.74x0.62mm_HandSolder -> Capacitor_SMD:C_0805_2012Metric_Pad1.18x1.45mm_HandSolder
- J1: footprint Connector_PinHeader_2.54mm:PinHeader_1x07_P2.54mm_Vertical -> Connector_PinSocket_2.54mm:PinSocket_1x04_P2.54mm_Vertical; moved to B.Cu
- R1, R2: value 1.5k -> 10k; footprint Resistor_SMD:R_0402_1005Metric_Pad0.72x0.64mm_HandSolder -> Resistor_SMD:R_0805_2012Metric_Pad1.20x1.40mm_HandSolder
- R3: value 1.5k -> 40k; footprint Resistor_SMD:R_0402_1005Metric_Pad0.72x0.64mm_HandSolder -> Resistor_SMD:R_0805_2012Metric_Pad1.20x1.40mm_HandSolder
- U1: value MSP430FR2433IRGET -> AS1115-BQFT; footprint Package_DFN_QFN:VQFN-24-1EP_4x4mm_P0.5mm_EP2.45x2.45mm -> Package_DFN_QFN:QFN-24-1EP_4x4mm_P0.5mm_EP2.7x2.7mm
- Y1: value 32.768kHz -> 32768Hz; footprint Crystal:Crystal_SMD_0603-2Pin_6.0x3.5mm_HandSoldering -> Crystal:Crystal_SMD_MicroCrystal_CC7V-T1A-2Pin_3.2x1.5mm_HandSoldering
- moved C1 100.0 mm to (218.9, 111.5), turned to 180 degrees
- moved BT1 94.4 mm to (207.5, 109.5)
- moved Y1 88.1 mm to (211.5, 100.8)
- moved R3 79.6 mm to (202.6, 118.8), turned to 180 degrees
- moved J1 75.4 mm to (204.0, 121.8), turned to 270 degrees
- moved R2 73.8 mm to (197.6, 102.4)
- moved U1 67.6 mm to (197.0, 109.2), turned to 270 degrees
- moved C2 62.5 mm to (219.0, 109.0), turned to 180 degrees
- moved C3 54.1 mm to (213.2, 98.7), turned to 180 degrees
- moved R1 50.1 mm to (197.6, 104.3)
Connections:
- C2 pad 1: XTAL_OUT -> +3V0
- C2 pad 2: Net-(C2-Pad2) -> GND
- C3 pad 1: XTAL_IN -> Net-(C3-Pad1)
- C3 pad 2: Net-(C3-Pad2) -> GND
- J1 pad 1: TST_SBWTCK -> Net-(D1-Pad2)
- J1 pad 2: RST_SBWTDIO -> TST_SBWTCK
- J1 pad 3: BCLUART_TXD -> RST_SBWTDIO
- J1 pad 4: BCLUART_RXD -> GND
- R1 pad 1: Net-(DIS1-Pad12) -> +3V0
- R1 pad 2: 7_SEG_A_A -> I2C_SDA
- R2 pad 1: Net-(DIS1-Pad11) -> +3V0
- R2 pad 2: 7_SEG_A_B -> I2C_SLC
- R3 pad 1: Net-(DIS1-Pad3) -> +3V0
- R3 pad 2: 7_SEG_A_C -> Net-(R3-Pad2)
- U1 pad 1: RST_SBWTDIO -> Net-(DISP1-Pad4)
- U1 pad 10: Net-(H1-Pad1) -> Net-(R3-Pad2)
- U1 pad 11: 7_SEG_A_A -> I2C_SLC
- U1 pad 12: 7_SEG_A_B -> Net-(DISP1-Pad12)
- U1 pad 13: 7_SEG_A_C -> Net-(DISP1-Pad9)
- U1 pad 14: 7_SEG_A_D -> Net-(DISP1-Pad11)
- U1 pad 15: 7_SEG_A_E -> Net-(DISP1-Pad7)
- U1 pad 16: 7_SEG_A_F -> +3V0
- U1 pad 17: 7_SEG_A_G -> Net-(DISP1-Pad3)
- U1 pad 19: 7_SEG_C_3 -> Net-(DISP1-Pad5)
- U1 pad 2: TST_SBWTCK -> Net-(DISP1-Pad6)
- U1 pad 20: 7_SEG_C_4 -> Net-(DISP1-Pad8)
- U1 pad 21: XTAL_OUT -> (no net)
- U1 pad 22: XTAL_IN -> I2C_SDA
- U1 pad 24: +3V0 -> Net-(DISP1-Pad10)
- U1 pad 3: BCLUART_TXD -> GND
- U1 pad 4: BCLUART_RXD -> (no net)
- U1 pad 5: 7_SEG_C_1 -> (no net)
- U1 pad 6: 7_SEG_C_2 -> (no net)
- U1 pad 7: Net-(H4-Pad1) -> (no net)
- U1 pad 8: Net-(H3-Pad1) -> (no net)
- U1 pad 9: Net-(H2-Pad1) -> (no net)
- Y1 pad 1: Net-(C2-Pad2) -> Net-(C4-Pad1)
- Y1 pad 2: Net-(C3-Pad2) -> Net-(C3-Pad1)
Routing:
- net +3V0: track 0.00 -> 71.1 mm, vias 0 -> 4
- net GND: track 0.00 -> 70.4 mm, vias 0 -> 3
- net Net-(DISP1-Pad9): track 0.00 -> 43.6 mm, vias 0 -> 2
- net TST_SBWTCK: track 0.00 -> 39.2 mm, vias 0 -> 1
- net Net-(DISP1-Pad11): track 0.00 -> 39.1 mm, vias 0 -> 2
- net Net-(DISP1-Pad7): track 0.00 -> 37.3 mm
- net RST_SBWTDIO: track 0.00 -> 32.9 mm, vias 0 -> 1
- net Net-(SW4-Pad1): track 0.00 -> 31.5 mm, vias 0 -> 2
- net Net-(SW3-Pad1): track 0.00 -> 31.0 mm, vias 0 -> 2
- net Net-(DISP1-Pad6): track 0.00 -> 27.0 mm, vias 0 -> 2
- net Net-(SW2-Pad1): track 0.00 -> 22.5 mm, vias 0 -> 1
- net Net-(SW1-Pad1): track 0.00 -> 22.2 mm, vias 0 -> 1
- net Net-(DISP1-Pad5): track 0.00 -> 21.9 mm, vias 0 -> 2
- net Net-(SW5-Pad1): track 0.00 -> 21.3 mm, vias 0 -> 1
- net I2C_SLC: track 0.00 -> 20.7 mm, vias 0 -> 2
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Other:
- board outline added: 29.5 x 29.5 mm
