File: sch/watch.kicad_pcb (KiCad board)
At the start: 4 copper layers, 29.5 x 29.5 mm, 19 parts, among them J1 eZ-FET, SW1 SW1, SW2 SW2, SW3 SW3, SW4 SW4, SW5 SW5, U1 AS1115-BQFT, U2 MSP430FR2433IRGET, Y1 32768Hz

Commit message: Added production files that was uploaded to JLCPCB.com
Parts:
- U1: value AS1115-BQFT -> AS1115
- U2: value MSP430FR2433IRGET -> MSP430FR2433
- renumbered DISP1 to Elektronika-1
Routing:
- net RST_SBWTDIO: track 32.9 -> 38.0 mm
- net Net-(DISP1-Pad8): track 17.9 -> 22.0 mm
- net Net-(DISP1-Pad9): track 43.8 -> 45.6 mm
- net Net-(DISP1-Pad4): track 17.6 -> 18.3 mm
- net Net-(DISP1-Pad12): track 18.9 -> 19.4 mm
- net Net-(SW3-Pad1): track 31.0 -> 31.5 mm
